File: schematics_and_pcbs/imac_g3_down_converter_board_adapter/imac_g3_down_converter_board_adapter.kicad_pcb (KiCad board)
At the start: 2 copper layers, 88 x 39 mm, 8 parts, among them J1 Screw_Terminal_01x10, J2 Screw_Terminal_01x04, J7 Conn_02x12_Top_Bottom, M1 Fan_Tacho_PWM

Commit message: graffittied silkscreens.
Other:
- net class Default removed
- board text added: "Matt Gray was here lol"
- board text added: "Rocky Hill Down converter breakout board Rev 1."
- board text added: "WayWayWay"
- board text added: "https://github.com/qbancoffee/imac_g3_ivad_board_init/"
- board text added: "trans rights!"
- board text removed: "Down converter break ouy board."
- board text removed: "Rev 1."
- board text removed: "Rocky HIll"
