File: schematics_and_pcbs/imac_g3_slot_loading_J22_adapter_board/imac_g3_slot_loading_J22_adapter_board.kicad_pcb (KiCad board)
At the start: 2 copper layers, 65 x 30 mm, 12 parts, among them J1 Conn_02x13_Odd_Even, J2 Screw_Terminal_01x10, J3 AudioJack3, J4 Conn_02x03_Odd_Even

Commit message: graffittied silkscreens.
Other:
- net class Default removed
- board text added: "Matt Gray was here lol"
- board text added: "Rocky Hill iMac G3 DV Adapter Board for Power Button, Speakers, LED & AC"
- board text added: "WayWayWay"
- board text added: "https://github.com/qbancoffee/imac_g3_ivad_board_init/"
- board text added: "trans rights!"
- board text removed: "iMac G3 DV Power Button / Speakers /LED's/ AC Adapter Board"
