File: schematics_and_pcbs/surfacemount_version/imac_g3_333mhz_slot_loading_J20_adapter_board/imac_g3_333mhz_slot_loading_J20_adapter_board.kicad_pcb (KiCad board)
At the start: 2 copper layers, 82.5 x 52.5 mm, 41 parts, among them J1 Screw_Terminal_01x06, J2 Conn_02x10_Odd_Even, J3 Conn_02x03_Odd_Even, J4 DE15_Receptacle_HighDensity_M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, J5 Conn_02x03_Odd_Even, J6 USB_C_Receptacle_USB2.0, U1 ATmega328P-AU, U2 TS5A23159DGS, U3 FT231XS, Y1 16 Mz cystal

Commit message: graffittied silkscreens.
Other:
- board text added: "Matt Gray was here lol"
- board text added: "WayWayWay"
- board text added: "https://github.com/qbancoffee/imac_g3_ivad_board_init"
- board text added: "trans rights!"
